File: pcb/circuit.brd (EAGLE design)
At the start: 80 x 80 mm, 149 parts, among them IC1 MCP73833-AMI/UN-ND, IC2 MCP3423, IC3 MCP1612-ADJI/MS, IC4 WE-TVS, IC5 ATWINC1510-MR210PB1952-ND, IC6 RN4870, IC7 MAX3378EEUD, IC8 ATSAML22N18A, J1 USB2-MICRO, J10 2.5MM-AUDIO-JACK-MONO, J11 2.5MM-AUDIO-JACK-MONONO_DRILL, J12 22-05-7028-02, J2 2.5MM-AUDIO-JACK-MONO, J3 2.5MM-AUDIO-JACK-MONONO_DRILL, J4 2.5MM-AUDIO-JACK-MONO, J5 2.5MM-AUDIO-JACK-MONONO_DRILL, J6 2.5MM-AUDIO-JACK-MONO, J7 2.5MM-AUDIO-JACK-MONONO_DRILL, J8 2.5MM-AUDIO-JACK-MONO, J9 2.5MM-AUDIO-JACK-MONONO_DRILL, Q1 ECX-1210, T1 PMOS, T10 NMOSSOT323, T11 NMOSSOT323, T12 NMOSSOT323, T13 NMOSSOT323, T2 PMOS, T3 NMOSSOT323, T4 NMOSSOT323, T5 NMOSSOT323, T6 NMOSSOT323, T7 NMOSSOT323, T8 NMOSSOT323, T9 NMOSSOT323, X1 LI-ION_BATHOL2, X2 B3S-1000, X3 MOLEX_1MM_FPC, X4 IGRID-20

Commit message: Board dimension created
-reworked schematics
-added PCB for battery-holder
-added PCB for UI
Parts:
- removed R20: 100k, rcl:R0603
- removed T2: PMOS, thermo:SOT23
- removed X1: LI-ION_BATHOL2, thermo:HOLDER_2
- added J13: 22-05-7038-03, con-molex:7395-03
- moved JP2 43.4 mm to (68.5, 30.8)
- moved JP1 28.8 mm to (38.5, 65.0)
- moved JP4 28.5 mm to (43.0, 65.0)
- moved J12 16.3 mm to (66.4, 40.0), turned to 90 degrees
- moved JP3 10.2 mm to (77.0, 70.1), turned to 90 degrees
- moved JP7 10.0 mm to (76.5, 60.3)
- moved JP6 9.50 mm to (71.0, 56.0)
- moved C26 9.33 mm to (-86.3, 142.6)
- moved IC1 9.22 mm to (32.0, 20.0), turned to 270 degrees
- moved IC5 8.10 mm to (29.6, 58.3), flipped to the bottom
- moved IC8 6.32 mm to (40.2, 37.2)
- moved IC6 4.90 mm to (55.0, 66.9), flipped to the bottom
- moved JP5 3.89 mm to (73.0, 64.3)
- moved X3 1.00 mm to (15.3, 22.8)
- moved X4 0.08 mm to (75.7, 25.0), flipped to the bottom, turned to 90 degrees
Connections:
- removed net POL_PROT_GATE: R20.2, T2.1
- net CHARGER_NTC: now also J13.2
- net GND: now also J13.3; no longer R20.1, X1.1, X1.3
- net VBAT: now also J13.1; no longer T2.2
- net VIN: no longer T2.3, X1.2, X1.4
Routing:
- net USB_D_N: track 8.33 -> 0.00 mm
- net USB_D_P: track 8.30 -> 0.00 mm
- net SENSOR_IN_9: track 0.00 -> 4.76 mm
- net SENSOR_IN_8: track 0.00 -> 4.76 mm
- net SENSOR_IN_7: track 0.00 -> 4.76 mm
- net SENSOR_IN_6: track 0.00 -> 4.76 mm
- net SENSOR_IN_5: track 0.00 -> 4.76 mm
- net USB_D_FIL_P: track 1.21 -> 0.00 mm
- net USB_D_FIL_N: track 1.21 -> 0.00 mm

Commit message: Routing
-routing 2.5mm Sensor Connectors started
Parts:
- moved R7 220.2 mm to (24.1, 26.8), flipped to the bottom, turned to 180 degrees
- moved R5 217.3 mm to (24.1, 24.7), flipped to the bottom, turned to 180 degrees
- moved R1 214.5 mm to (24.1, 22.6), flipped to the bottom, turned to 180 degrees
- moved J13 59.6 mm to (13.7, 19.4), turned to 270 degrees
- moved SV1 10.0 mm to (4.97, 40.2)
- moved D1 8.38 mm to (21.0, 22.6), turned to 0 degrees
- moved X3 8.06 mm to (14.3, 30.8)
- moved D3 7.83 mm to (21.0, 26.8), turned to 0 degrees
- moved D2 7.03 mm to (21.0, 24.7), turned to 0 degrees
- moved IC1 2.24 mm to (30.0, 19.0)
Routing:
- net SENSOR_EN_1: track 0.00 -> 9.94 mm
- net SENSOR_IN_0_DRAIN: track 0.00 -> 7.76 mm
- net SENSOR_EN_0: track 0.00 -> 7.47 mm
- net CHARGER_STAT2_LED: track 0.00 -> 1.25 mm
- net CHARGER_STAT1_LED: track 0.00 -> 1.25 mm
- net CHARGER_!PG!_LED: track 0.00 -> 1.25 mm

Commit message: Power Unit
- placed power devices
Parts:
- removed R58: 1M, rcl:R0603
- removed T13: NMOSSOT323, Thermo_Library:SOT-323
- removed X4: IGRID-20, thermo:I-GRID-20
- added C22: 10µF, rcl:C0805
- added R20: 330, rcl:R0603
- added T2: NMOSSOT323, Thermo_Library:SOT-323
- added X1: B3S-1000, Thermo_Library:B3S
- C10, C27: value 1nF -> 10µF; device rcl:C0603 -> rcl:C0805
- C11: value 4,7nF -> 100nF
- C12, C28: value 100nF -> 1nF
- C17, C18: value 10µF -> 100nF; device rcl:C0805 -> rcl:C0603
- C20, C32, C37: value 100nF -> 1µF
- C21, C34: value 100nF -> 10µF; device rcl:C0603 -> rcl:C0805
- C23, C33: value 1µF -> 100nF
- C24, C25: value 22pF -> 100nF
- C29: value 10µF -> 1µF; device rcl:C0805 -> rcl:C0603
- C30: value 10µF -> 1nF; device rcl:C0805 -> rcl:C0603
- C31: value 1nF -> 100nF
- C35, C36: value 1µF -> 22pF
- C9: value 100nF -> 4,7nF
- IC1: value MCP73833-AMI/UN-ND -> MCP1612-ADJI/MS; device thermo:MSOP10 -> thermo:MSOP8
- IC2: value MCP3423 -> MCP73833-AMI/UN-ND
- IC3: value MCP1612-ADJI/MS -> WE-TVS; device thermo:MSOP8 -> thermo:SOT23-5L
- IC4: value WE-TVS -> MCP3423; device thermo:SOT23-5L -> thermo:MSOP10
- IC6: value RN4870 -> MAX3378EEUD; device thermo:RN4870-MODULE -> thermo:TSSOP14
- IC7: value MAX3378EEUD -> RN4870; device thermo:TSSOP14 -> thermo:RN4870-MODULE
- J1: value USB2-MICRO -> 22-05-7038-03; device thermo:USB-2-MICRO -> con-molex:7395-03
- J10: value 2.5MM-AUDIO-JACK-MONO -> 2.5MM-AUDIO-JACK-MONONO_DRILL; device Thermo_Library:2.5MM-AUDIO-JACK-MONO -> thermo:2.5MM-AUDIO-JACK-MONO-2
- J12: value 22-05-7028-02 -> 2.5MM-AUDIO-JACK-MONONO_DRILL; device con-molex:7395-02 -> thermo:2.5MM-AUDIO-JACK-MONO-2
- J13: value 22-05-7038-03 -> 2.5MM-AUDIO-JACK-MONONO_DRILL; device con-molex:7395-03 -> thermo:2.5MM-AUDIO-JACK-MONO-2
- J2: value 2.5MM-AUDIO-JACK-MONO -> USB2-MICRO; device Thermo_Library:2.5MM-AUDIO-JACK-MONO -> thermo:USB-2-MICRO
- J3, J5, J7: value 2.5MM-AUDIO-JACK-MONONO_DRILL -> 2.5MM-AUDIO-JACK-MONO; device thermo:2.5MM-AUDIO-JACK-MONO-2 -> Thermo_Library:2.5MM-AUDIO-JACK-MONO
- J8: value 2.5MM-AUDIO-JACK-MONO -> 22-05-7028-02; device Thermo_Library:2.5MM-AUDIO-JACK-MONO -> con-molex:7395-02
- JP3: value 3 -> 2; device jumper:JP2 -> jumper:JP1
- JP4: value 4 -> 2; device jumper:JP4 -> jumper:JP1
- JP5: value 2 -> 3; device jumper:JP1 -> jumper:JP2
- JP6: value 2 -> 4; device jumper:JP1 -> jumper:JP4
- L4: value 10µH -> (none); device Thermo_Library:L-1210 -> Thermo_Library:L0603
- L5: value (none) -> 10µH; device Thermo_Library:L0603 -> Thermo_Library:L-1210
- R1: value 270 -> 10
- R10: value 2.2M -> 0
- R11: value 1.8M -> 301k
- R12: value 301k -> 324k
- R14: value 10 -> 100m; device rcl:R0603 -> rcl:R5025
- R15: value 324k -> 2.2M
- R16: value 25k -> 1M; device rcl:R0805 -> rcl:R0603
- R17: value 200k -> 1.8M
- R18: value 0 -> 4,7k
- R19: value 1M -> 4,7k
- R2: value 4,7k -> 25k; device rcl:R0603 -> rcl:R0805
- R21, R22: value 0 -> 1M
- R23: value 0 -> 10k
- R26, R31: value 1M -> 0
- R3: value 4,7k -> 270
- R32: value 4,7k -> 0
- R36: value 10k -> 4,7k
- R37: value 330 -> 1M
- R4: value 100m -> 270; device rcl:R5025 -> rcl:R0603
- R43, R44, R45, R46, R47: value 4.7k 0.1% -> 1M
- R48, R49, R50, R51, R52: value 1M -> 4.7k 0.1%
- R6: value 1.54k -> 200k
- R7: value 270 -> 2k
- R8: value 2k -> 1.54k
- X2: value B3S-1000 -> MOLEX_1MM_FPC; device Thermo_Library:B3S -> thermo:1MM_FPC_ZIF
- X3: value MOLEX_1MM_FPC -> IGRID-20; device thermo:1MM_FPC_ZIF -> thermo:I-GRID-20
- moved R37 276.2 mm to (71.5, 7.20), flipped to the bottom, turned to 90 degrees
- moved C7 262.8 mm to (59.2, 17.9), flipped to the bottom, turned to 90 degrees
- moved L4 256.8 mm to (-137.2, 158.8), turned to 0 degrees
- moved L5 256.8 mm to (119.4, 170.2), turned to 270 degrees
- moved C36 249.4 mm to (108.5, 179.2), turned to 90 degrees
- moved C35 247.3 mm to (111.5, 179.2), turned to 90 degrees
- moved C4 243.2 mm to (46.0, 25.6), flipped to the bottom
- moved C20 240.6 mm to (-134.6, 154.9)
- moved R12 230.5 mm to (51.0, 21.1), flipped to the bottom, turned to 90 degrees
- moved R57 229.5 mm to (-104.1, 154.9), flipped to the top, turned to 0 degrees
- moved T12 228.5 mm to (-109.2, 158.8), flipped to the top, turned to 0 degrees
- moved C1 227.9 mm to (34.3, 11.8), flipped to the bottom, turned to 90 degrees
- moved R11 226.9 mm to (53.0, 21.1), flipped to the bottom, turned to 270 degrees
- moved R17 217.0 mm to (21.0, 19.6), flipped to the bottom, turned to 90 degrees
- moved C6 216.5 mm to (57.1, 17.9), flipped to the bottom, turned to 90 degrees
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Connections:
- net !OLED_RESET: now also X3.16; no longer X4.16
- net !OLED_SPI_CS: now also X3.17; no longer X4.17
- net !PG!_TRANS: now also IC6.2; no longer IC7.2
- net !RESET!: now also C15.1, R20.2, R23.1; no longer C37.1, R36.1, R37.2
- net !RESET!_B: now also R20.1, X1.2, X1.4; no longer R37.1, X2.2, X2.4
- net +3V3: now also C10.1, C11.1, C18.1, C19.1, C20.1, C21.1, C30.1, C33.1, IC4.6, IC6.1, IC7.4, IC7.6, IC7.7, L4.2, R11.2, R18.2, R19.2, R23.2, R34.2, R35.2, X2.1, X2.7, X3.2; no longer C15.1, C2.1, C26.1, C28.1, C29.1, C3.1, C35.1, C4.1, IC2.6, IC6.4, IC6.6, IC6.7, IC7.1, J10.2, J11.2, J2.2, J3.2, J4.2, J5.2, J6.2, J7.2, J8.2, J9.2, L5.2, R12.2, R2.2, R26.2, R3.2, R31.2, R32.2, X3.1, X3.7, X4.2
- net +3V3_ANA: now also C22.1, C23.1, C24.1, J10.2, J11.2, J12.2, J13.2, J3.2, J4.2, J5.2, J6.2, J7.2, J9.2, L4.1; no longer C18.1, C19.1, C20.1, L5.1
- net AD_CH2+: now also IC4.4, R15.2, R17.2; no longer IC2.4, R10.2, R11.2
- net AD_SCL: now also IC4.8, JP3.1, R18.1; no longer IC2.8, JP5.1, R2.1
- net AD_SDA: now also IC4.7, JP3.2, R19.1; no longer IC2.7, JP5.2, R3.1
- net AGND: now also C22.2, C23.2, C24.2, C25.2, C3.2, C4.1, IC1.6, R10.2, R13.1, R6.1, T2.2; no longer C10.1, C11.2, C18.2, C19.2, C20.2, C21.2, IC3.6, R17.1, R18.2, R19.1, T12.2
- net BT_!RESET!: now also C37.1, IC7.21, R36.1; no longer C33.1, IC6.21, R32.1
- net BT_LINK_DROP: now also IC7.25; no longer IC6.25
- net BT_MODE: now also IC7.18, R35.1; no longer IC6.18, R31.1
- net BT_PAIRING_KEY: now also IC7.27; no longer IC6.27
- net BT_RSSI_IND: now also IC7.24; no longer IC6.24
- net BT_RX_IND: now also IC7.26; no longer IC6.26
- net BT_STATUS_1: now also IC7.12; no longer IC6.12
- net BT_STATUS_2: now also IC7.16; no longer IC6.16
- net BT_TX_IND: now also IC7.11; no longer IC6.11
- net BT_UART_CTS: now also IC7.15, JP6.2; no longer IC6.15, JP4.2
- net BT_UART_RTS: now also IC7.17, JP6.1; no longer IC6.17, JP4.1
- net BT_UART_RX: now also IC7.22, JP6.4; no longer IC6.22, JP4.4
- net BT_UART_TX: now also IC7.23, JP6.3; no longer IC6.23, JP4.3
- net BUCK_FB: now also IC1.5, R12.1, R6.2; no longer IC3.5, R15.1, R17.2
- net BUCK_FB_R: now also R11.1, R12.2; no longer R12.1, R15.2
- net BUCK_LX: now also IC1.8; no longer IC3.8
- net BUCK_RC_C: now also C4.2, R2.2; no longer C10.2, R16.2
- net BUCK_RC_R: now also IC1.4, R2.1; no longer IC3.4, R16.1
- net BUCK_V+: now also C2.1, IC1.1, IC1.3, R1.2; no longer C8.1, IC3.1, IC3.3, R14.2
- net BUCK_VCC: now also C3.1, IC1.2, R1.1; no longer C9.1, IC3.2, R14.1
- net CHARGER_!PG!: now also IC2.7, IC6.13, R5.2; no longer IC1.7, IC7.13, R7.2
- net CHARGER_!PG!_LED: now also R5.1; no longer R7.1
- net CHARGER_NTC: now also J1.2, R8.1; no longer J13.2, R6.1
- net CHARGER_PROG: now also IC2.6, R7.2; no longer IC1.6, R8.2
- net CHARGER_STAT1: now also IC2.3, IC6.11, R3.2; no longer IC1.3, IC7.11, R1.2
- net CHARGER_STAT1_LED: now also R3.1; no longer R1.1
- net CHARGER_STAT2: now also IC2.4, IC6.12, R4.2; no longer IC1.4, IC7.12, R5.2
- net CHARGER_STAT2_LED: now also R4.1; no longer R5.1
- net CHARGER_THERM: now also IC2.8, R8.2; no longer IC1.8, R6.2
- net CHARGER_VBAT_MEAS: now also C8.1, IC2.10, IC2.9, IC4.2, R14.2; no longer C1.1, IC1.10, IC1.9, IC2.2, R4.2
- net CHARGER_VUSB_FIL: now also C1.1, C32.1, IC2.1, IC2.2, IC3.5, IC6.10, IC6.14, IC6.8, R16.2; no longer C36.1, IC1.1, IC1.2, IC4.5, IC7.10, IC7.14, IC7.8, R13.2
- net EXT_PWM_0: now also J8.1; no longer J12.1
- net EXT_PWM_1: now also J8.2; no longer J12.2
- net GND: now also C10.2, C11.2, C18.2, C19.2, C20.2, C21.2, IC1.7, IC3.2, IC4.10, IC4.3, IC4.5, IC4.9, IC6.7, IC7.1, IC7.2, IC7.3, IC7.31, IC7.32, IC7.33, J1.3, J2.5, R10.1, R16.1, R17.1, R21.1, R22.1, R37.1, R43.1, R44.1, R45.1, R46.1, R47.1, R7.1, T12.2, X1.1, X1.3, X2.12, X2.6; no longer C23.2, C24.2, C25.2, C3.2, C4.2, IC1.5, IC2.10, IC2.3, IC2.9, IC3.7, IC4.2, IC6.1, IC6.2, IC6.3, IC6.31, IC6.32, IC6.33, IC7.7, J1.5, J13.3, R11.1, R13.1, R18.1, R34.1, R35.1, R48.1, R49.1, R50.1, R51.1, R52.1, R58.1, R8.1, T13.2, X2.1, X2.3, X3.12, X3.6
- net OLED_D/C: now also X3.4; no longer X4.4
- net OLED_EN: now also R57.2, T12.1; no longer R58.2, T13.1
- net OLED_EN_DRAIN: now also T12.3, X3.1, X3.10, X3.11, X3.12, X3.13, X3.14, X3.19, X3.20, X3.5, X3.6; no longer T13.3, X4.1, X4.10, X4.11, X4.12, X4.13, X4.14, X4.19, X4.20, X4.5, X4.6
- net OLED_SPI_MOSI: now also X3.8; no longer X4.8
- net OLED_SPI_SCLK: now also X3.7; no longer X4.7
- net RES0: now also JP5.1; no longer JP3.1
- net RES1: now also JP5.2; no longer JP3.2
- net RES2: now also JP5.3; no longer JP3.3
- net SENSOR_EN_0: now also R37.2, T2.1; no longer R48.2, T3.1
- net SENSOR_EN_1: now also R43.2, T3.1; no longer R49.2, T5.1
- net SENSOR_EN_2: now also R44.2, T4.1; no longer R50.2, T7.1
- net SENSOR_EN_3: now also R45.2, T5.1; no longer R51.2, T9.1
- net SENSOR_EN_4: now also R46.2, T6.1; no longer R52.2, T11.1
- net SENSOR_EN_5: now also R47.2, T7.1; no longer R53.2, T4.1
- net SENSOR_EN_6: now also R53.2, T8.1; no longer R54.2, T6.1
- net SENSOR_EN_7: now also R54.2, T9.1; no longer R55.2, T8.1
- net SENSOR_EN_8: now also R55.2; no longer R56.2
- net SENSOR_EN_9: now also R56.2, T11.1; no longer R57.2, T12.1
- net SENSOR_INT_0: now also J3.3; no longer J2.3
- net SENSOR_INT_2: now also J5.3; no longer J6.3
- net SENSOR_INT_3: now also J6.3; no longer J8.3
- net SENSOR_INT_4: now also J7.3; no longer J10.3
- net SENSOR_INT_5: now also J9.3; no longer J3.3
- net SENSOR_INT_6: now also J10.3; no longer J5.3
- net SENSOR_INT_7: now also J11.3; no longer J7.3
- net SENSOR_INT_8: now also J12.3; no longer J9.3
- net SENSOR_INT_9: now also J13.3; no longer J11.3
- net SENSOR_IN_0: now also J3.1; no longer J2.1
- net SENSOR_IN_0_DRAIN: now also T2.3; no longer T3.3
- net SENSOR_IN_1: now also R39.1; no longer R40.1
- net SENSOR_IN_1_DRAIN: now also R39.2, T3.3; no longer R40.2, T5.3
- net SENSOR_IN_2: now also J5.1, R40.1; no longer J6.1, R42.1
- net SENSOR_IN_2_DRAIN: now also R40.2, T4.3; no longer R42.2, T7.3
- net SENSOR_IN_3: now also J6.1, R41.1; no longer J8.1, R44.1
- net SENSOR_IN_3_DRAIN: now also R41.2, T5.3; no longer R44.2, T9.3
- net SENSOR_IN_4: now also J7.1, R42.1; no longer J10.1, R46.1
- net SENSOR_IN_4_DRAIN: now also R42.2, T6.3; no longer R46.2, T11.3
- net SENSOR_IN_5: now also J9.1, R48.1; no longer J3.1, R39.1
- net SENSOR_IN_5_DRAIN: now also R48.2, T7.3; no longer R39.2, T4.3
- net SENSOR_IN_6: now also J10.1, R49.1; no longer J5.1, R41.1
- net SENSOR_IN_6_DRAIN: now also R49.2, T8.3; no longer R41.2, T6.3
- net SENSOR_IN_7: now also J11.1, R50.1; no longer J7.1, R43.1
- net SENSOR_IN_7_DRAIN: now also R50.2, T9.3; no longer R43.2, T8.3
- net SENSOR_IN_8: now also J12.1, R51.1; no longer J9.1, R45.1
- net SENSOR_IN_8_DRAIN: now also R51.2; no longer R45.2
- net SENSOR_IN_9: now also J13.1, R52.1; no longer J11.1, R47.1
- net SENSOR_IN_9_DRAIN: now also R52.2, T11.3; no longer R47.2, T12.3
- net STAT1_TRANS: now also IC6.4; no longer IC7.4
- net STAT2_TRANS: now also IC6.3; no longer IC7.3
- net UI_BUTTON_INT_0: now also X2.2, X2.8; no longer X3.2, X3.8
- net UI_BUTTON_INT_1: now also X2.3, X2.9; no longer X3.3, X3.9
- net UI_BUTTON_INT_2: now also X2.10, X2.4; no longer X3.10, X3.4
- net UI_BUTTON_INT_3: now also X2.11, X2.5; no longer X3.11, X3.5
- net USB_CON_INT_TRANS: now also IC6.5; no longer IC7.5
- net USB_D_N: now also IC3.3, J2.2; no longer IC4.3, J1.2
- net USB_D_P: now also IC3.4, J2.3; no longer IC4.4, J1.3
- net USB_SHIELD: now also C9.1, J2.6, J2.7, J2.8, J2.9, R13.2; no longer C11.1, J1.6, J1.7, J1.8, J1.9, R19.2
- net USB_VCC: now also J2.1; no longer J1.1
- net VBAT: now also IC4.1, J1.1, R14.1, R15.1; no longer IC2.1, J13.1, R10.1, R4.1
- net VDDCORE: now also C25.1, C29.1, L5.2; no longer C21.1, C23.1, L4.2
- net VDDOUT: now also L5.1; no longer L4.1
- net WIFI_1P3V_TP: now also C26.1, C28.1; no longer C30.1, C32.1
- net WIFI_CHIP_EN: now also R32.1; no longer R30.1
- net WIFI_CHIP_EN_D: now also R22.2, R32.2; no longer R30.2, R35.2
- net WIFI_IRQN: now also R25.1; no longer R22.1
- net WIFI_IRQN_D: now also R25.2; no longer R22.2
- net WIFI_RESETN_D: now also R21.2; no longer R34.2
- net WIFI_SPI_CFG: now also R34.1; no longer R26.1
- net WIFI_SPI_MISO: now also R29.1; no longer R27.1
- net WIFI_SPI_MISO_D: now also R29.2; no longer R27.2
- net WIFI_SPI_MOSI: now also R27.1; no longer R24.1
- net WIFI_SPI_MOSI_D: now also R27.2; no longer R24.2
- net WIFI_SPI_SCK: now also R30.1; no longer R28.1
- net WIFI_SPI_SCK_D: now also R30.2; no longer R28.2
- net WIFI_SPI_SSN: now also R28.1; no longer R25.1
- net WIFI_SPI_SSN_D: now also R28.2; no longer R25.2
- net WIFI_UART1_RXD: now also JP4.2, R31.1; no longer JP6.2, R29.1
- net WIFI_UART1_RXD_D: now also R31.2; no longer R29.2
- net WIFI_UART1_TXD: now also JP4.1, R26.1; no longer JP6.1, R23.1
- net WIFI_UART1_TXD_D: now also R26.2; no longer R23.2
- net WIFI_WAKE: now also R24.1; no longer R21.1
- net WIFI_WAKE_D: now also R24.2; no longer R21.2
- net XIN32: now also C35.1; no longer C24.1
- net XOUT32: now also C36.1; no longer C25.1
Routing:
- net CHARGER_VUSB_FIL: track 0.00 -> 28.5 mm, vias 0 -> 1
- net CHARGER_VBAT_MEAS: track 0.00 -> 24.5 mm
- net GND: track 0.93 -> 22.0 mm
- net SENSOR_EN_4: track 0.00 -> 10.2 mm
- net SENSOR_EN_2: track 0.00 -> 10.1 mm
- net SENSOR_EN_9: track 0.00 -> 10.0 mm
- net SENSOR_EN_8: track 0.00 -> 10.0 mm
- net SENSOR_EN_7: track 0.00 -> 10.0 mm
- net SENSOR_EN_6: track 0.00 -> 10.0 mm
- net SENSOR_EN_5: track 0.00 -> 10.0 mm
- net SENSOR_EN_3: track 0.00 -> 10.0 mm
- net BUCK_V+: track 0.00 -> 8.57 mm
- net SENSOR_IN_5_DRAIN: track 0.00 -> 7.94 mm
- net SENSOR_IN_8_DRAIN: track 0.00 -> 7.94 mm
- net SENSOR_IN_6_DRAIN: track 0.00 -> 7.94 mm
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
Commit message: AD Converter placed
Parts:
- R21, R22: value 1M -> 0
- R23: value 10k -> 0
- R31: value 0 -> 10k
- R32, R33: value 0 -> 1M
- moved R23 397.9 mm to (233.9, 206.2), flipped to the bottom
- moved L4 230.0 mm to (48.6, 23.1), flipped to the bottom
- moved T12 224.6 mm to (71.8, 25.8)
- moved R57 221.8 mm to (73.4, 21.9), turned to 270 degrees
- moved R20 208.7 mm to (14.6, 43.6), flipped to the bottom, turned to 270 degrees
- moved C37 205.5 mm to (50.4, 55.5), flipped to the bottom, turned to 270 degrees
- moved C32 201.0 mm to (14.0, 25.4), flipped to the bottom, turned to 180 degrees
- moved C20 191.2 mm to (14.0, 34.7), flipped to the bottom
- moved R26 188.5 mm to (233.9, 200.1)
- moved R25 181.3 mm to (233.9, 202.2)
- moved R10 181.1 mm to (48.6, 21.1), flipped to the bottom, turned to 180 degrees
- moved R28 181.0 mm to (233.9, 196.0)
- moved R27 179.1 mm to (233.9, 198.1)
- moved R24 178.9 mm to (233.9, 204.2), flipped to the bottom
- moved R22 178.0 mm to (233.9, 208.3)
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Connections:
- removed net WIFI_SPI_MOSI_D: IC5.15, R27.2
- removed net WIFI_UART1_TXD_D: IC5.14, R26.2
- new net WIFI_MOSI_D: IC5.15, R24.2
- new net WIFI_UART_TXD_D: IC5.14, R23.2
- net !RESET!: now also R31.1; no longer R23.1
- net +3V3: now also R31.2; no longer R23.2
- net AD_CH2+: now also IC4.1; no longer IC4.4
- net CHARGER_VBAT_MEAS: now also IC4.5; no longer IC4.2
- net GND: now also IC4.2, R32.1, R33.1; no longer IC4.5, R21.1, R22.1
- net VBAT: now also IC4.4; no longer IC4.1
- net WIFI_CHIP_EN: now also R29.1; no longer R32.1
- net WIFI_CHIP_EN_D: now also R29.2, R33.2; no longer R22.2, R32.2
- net WIFI_IRQN: now also R22.1; no longer R25.1
- net WIFI_IRQN_D: now also R22.2; no longer R25.2
- net WIFI_RESETN: now also R30.1; no longer R33.1
- net WIFI_RESETN_D: now also R30.2, R32.2; no longer R21.2, R33.2
- net WIFI_SPI_MISO: now also R26.1; no longer R29.1
- net WIFI_SPI_MISO_D: now also R26.2; no longer R29.2
- net WIFI_SPI_MOSI: now also R24.1; no longer R27.1
- net WIFI_SPI_SCK: now also R27.1; no longer R30.1
- net WIFI_SPI_SCK_D: now also R27.2; no longer R30.2
- net WIFI_SPI_SSN: now also R25.1; no longer R28.1
- net WIFI_SPI_SSN_D: now also R25.2; no longer R28.2
- net WIFI_UART1_RXD: now also R28.1; no longer R31.1
- net WIFI_UART1_RXD_D: now also R28.2; no longer R31.2
- net WIFI_UART1_TXD: now also R23.1; no longer R26.1
- net WIFI_WAKE: now also R21.1; no longer R24.1
- net WIFI_WAKE_D: now also R21.2; no longer R24.2
Routing:
- net GND: track 22.0 -> 240.6 mm, vias 0 -> 1
- net CHARGER_VUSB_FIL: track 28.5 -> 78.7 mm, vias 1 -> 3
- net +3V3: track 5.60 -> 41.8 mm
- net VBAT: track 4.39 -> 20.8 mm
- net CHARGER_STAT1: track 0.00 -> 13.2 mm
- net WIFI_CHIP_EN_D: track 0.00 -> 13.2 mm
- net CHARGER_!PG!: track 0.00 -> 12.5 mm, vias 0 -> 2
- net CHARGER_STAT2: track 0.00 -> 10.3 mm
- net !RESET!_B: track 0.00 -> 9.59 mm
- net CHARGER_NTC: track 2.05 -> 9.10 mm
- net WIFI_1P3V_TP: track 0.00 -> 6.79 mm
- net BUCK_V+: track 8.57 -> 14.4 mm
- net AD_CH2+: track 0.00 -> 4.59 mm
- net WIFI_RESETN_D: track 0.00 -> 4.34 mm
- net USB_D_FIL_N: track 1.88 -> 6.04 mm
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
Commit message: Power Unit Refactored
Parts:
- moved R21 428.4 mm to (-194.1, 192.3)
- moved R22 428.4 mm to (-194.1, 190.3)
- moved R23 428.4 mm to (-194.1, 188.2)
- moved R24 428.4 mm to (-194.1, 186.2)
- moved R25 428.4 mm to (-194.1, 184.2)
- moved R26 428.4 mm to (-194.1, 182.1)
- moved R27 428.4 mm to (-194.1, 180.1)
- moved R28 428.4 mm to (-194.1, 178.0)
- moved R34 428.4 mm to (-194.1, 194.4)
- moved JP1 236.8 mm to (-165.8, 27.5)
- moved JP2 236.8 mm to (-162.0, 19.0)
- moved JP5 236.8 mm to (-157.0, 41.1)
- moved JP6 236.8 mm to (-170.0, 19.0)
- moved JP7 236.8 mm to (-157.5, 31.3)
- moved C13 216.6 mm to (-123.0, 64.7)
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Routing:
- net GND: track 240.6 -> 137.3 mm, vias 1 -> 2
- net CHARGER_VUSB_FIL: track 78.7 -> 26.2 mm, vias 3 -> 1
- net CHARGER_NTC: track 9.10 -> 26.1 mm
- net CHARGER_STAT1: track 13.2 -> 0.00 mm
- net CHARGER_!PG!: track 12.5 -> 0.00 mm, vias 2 -> 0
- net CHARGER_STAT2: track 10.3 -> 0.00 mm
- net VBAT: track 20.8 -> 12.3 mm
- net CHARGER_VBAT_MEAS: track 26.6 -> 18.3 mm
- net AGND: track 8.38 -> 3.50 mm
- net USB_D_FIL_N: track 6.04 -> 2.11 mm
- net USB_D_FIL_P: track 5.56 -> 1.95 mm
- net BUCK_LX: track 2.67 -> 6.25 mm
- net CHARGER_THERM: track 3.59 -> 6.64 mm, vias 1 -> 0
- net USB_SHIELD: track 4.89 -> 2.10 mm
- net BUCK_VCC: track 3.82 -> 6.39 mm
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
Commit message: Power Unit
-power unit routed
Parts:
- removed J10, J11, J12, J13: 2.5MM-AUDIO-JACK-MONONO_DRILL, thermo:2.5MM-AUDIO-JACK-MONO-2
- removed J3, J4, J5, J6, J7: 2.5MM-AUDIO-JACK-MONO, Thermo_Library:2.5MM-AUDIO-JACK-MONO
- removed J8: 22-05-7028-02, con-molex:7395-02
- removed SV1: JTAGEDU, con-harting-ml:ML20
- removed X3: IGRID-20, thermo:I-GRID-20
- added U$1: JTAG-EDGE-CON, thermo:DEBUG-CON
- added X10, X11, X12, X13: 2.5MM-AUDIO-JACK-MONONO_DRILL, thermo:2.5MM-AUDIO-JACK-MONO-2
- added X14: MOLEX_1MM_FPC, thermo:1MM_FPC_ZIF
- added X15: IGRID-20, thermo:I-GRID-20
- added X4, X5, X6, X7, X8: 2.5MM-AUDIO-JACK-MONODRILL, thermo:2.5MM-AUDIO-JACK-MONO
- C32: value 1µF -> 100nF
- C33: value 100nF -> 1µF
- J2: value USB2-MICRO -> 22-05-7038-03; device thermo:USB-2-MICRO -> con-molex:7395-03
- JP1, JP2, JP6, JP7: value 4 -> (none); device jumper:JP4 -> thermo:JP4
- JP3, JP4: value 2 -> (none); device jumper:JP1 -> thermo:JP2
- JP5: value 3 -> (none); device jumper:JP2 -> thermo:JP3
- X1: value B3S-1000 -> USB2-MICRO; device Thermo_Library:B3S -> thermo:USB-2-MICRO
- X2: value MOLEX_1MM_FPC -> B3S-1000; device thermo:1MM_FPC_ZIF -> Thermo_Library:B3S
- moved X2 187.5 mm to (69.5, 4.35), turned to 0 degrees
- moved JP3 170.7 mm to (-216.0, 5.00), turned to 0 degrees
- moved JP4 168.4 mm to (-230.0, 5.00), flipped to the top, turned to 0 degrees
- moved R57 158.0 mm to (32.6, 11.9), turned to 0 degrees
- moved C25 156.5 mm to (54.4, 39.9), turned to 90 degrees
- moved T12 155.3 mm to (32.6, 10.3)
- moved C23 155.0 mm to (32.6, 48.9), turned to 90 degrees
- moved C29 155.0 mm to (52.4, 39.9)
- moved C14 154.8 mm to (31.1, 32.0)
- moved C16 154.7 mm to (39.8, 29.5)
- moved Q1 154.7 mm to (45.8, 49.9)
- moved C36 154.6 mm to (44.2, 52.1)
- moved C17 154.6 mm to (48.9, 32.0)
- moved C35 154.6 mm to (47.2, 52.1)
- moved C24 154.6 mm to (40.8, 50.5)
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- renumbered J9 to X9
Connections:
- net !OLED_RESET: now also X15.16; no longer X3.16
- net !OLED_SPI_CS: now also X15.17; no longer X3.17
- net !RESET!: now also U$1.9; no longer SV1.15
- net !RESET!_B: now also X2.2, X2.4; no longer X1.2, X1.4
- net +3V3: now also C32.1, U$1.1, X14.1, X14.7, X15.2; no longer C33.1, SV1.1, X2.1, X2.7, X3.2
- net +3V3_ANA: now also X10.2, X11.2, X12.2, X13.2, X4.2, X5.2, X6.2, X7.2, X8.2; no longer J10.2, J11.2, J12.2, J13.2, J3.2, J4.2, J5.2, J6.2, J7.2
- net CHARGER_STAT1: now also IC6.12; no longer IC6.11
- net CHARGER_STAT2: now also IC6.11; no longer IC6.12
- net CHARGER_VUSB_FIL: now also C33.1; no longer C32.1
- net EXT_PWM_0: now also J2.1; no longer J8.1
- net EXT_PWM_1: now also J2.2; no longer J8.2
- net GND: now also J2.3, U$1.10, U$1.2, U$1.4, U$1.6, U$1.8, X1.5, X14.12, X14.6, X2.1, X2.3; no longer J2.5, SV1.10, SV1.12, SV1.14, SV1.16, SV1.18, SV1.20, SV1.4, SV1.6, SV1.8, X1.1, X1.3, X2.12, X2.6
- net OLED_D/C: now also X15.4; no longer X3.4
- net OLED_EN_DRAIN: now also X15.1, X15.10, X15.11, X15.12, X15.13, X15.14, X15.19, X15.20, X15.5, X15.6; no longer X3.1, X3.10, X3.11, X3.12, X3.13, X3.14, X3.19, X3.20, X3.5, X3.6
- net OLED_SPI_MOSI: now also X15.8; no longer X3.8
- net OLED_SPI_SCLK: now also X15.7; no longer X3.7
- net SENSOR_INT_0: now also X4.3; no longer J3.3
- net SENSOR_INT_1: now also X5.3; no longer J4.3
- net SENSOR_INT_2: now also X6.3; no longer J5.3
- net SENSOR_INT_3: now also X7.3; no longer J6.3
- net SENSOR_INT_4: now also X8.3; no longer J7.3
- net SENSOR_INT_6: now also X10.3; no longer J10.3
- net SENSOR_INT_7: now also X11.3; no longer J11.3
- net SENSOR_INT_8: now also X12.3; no longer J12.3
- net SENSOR_INT_9: now also X13.3; no longer J13.3
- net SENSOR_IN_0: now also X4.1; no longer J3.1
- net SENSOR_IN_1: now also X5.1; no longer J4.1
- net SENSOR_IN_2: now also X6.1; no longer J5.1
- net SENSOR_IN_3: now also X7.1; no longer J6.1
- net SENSOR_IN_4: now also X8.1; no longer J7.1
- net SENSOR_IN_6: now also X10.1; no longer J10.1
- net SENSOR_IN_7: now also X11.1; no longer J11.1
- net SENSOR_IN_8: now also X12.1; no longer J12.1
- net SENSOR_IN_9: now also X13.1; no longer J13.1
- net STAT1_TRANS: now also IC6.3; no longer IC6.4
- net STAT2_TRANS: now also IC6.4; no longer IC6.3
- net SWDCLK: now also U$1.5; no longer SV1.9
- net SWDIO: now also U$1.3; no longer SV1.7
- net UI_BUTTON_INT_0: now also X14.2, X14.8; no longer X2.2, X2.8
- net UI_BUTTON_INT_1: now also X14.3, X14.9; no longer X2.3, X2.9
- net UI_BUTTON_INT_2: now also X14.10, X14.4; no longer X2.10, X2.4
- net UI_BUTTON_INT_3: now also X14.11, X14.5; no longer X2.11, X2.5
- net USB_D_N: now also X1.2; no longer J2.2
- net USB_D_P: now also X1.3; no longer J2.3
- net USB_SHIELD: now also X1.6, X1.7, X1.8, X1.9; no longer J2.6, J2.7, J2.8, J2.9
- net USB_VCC: now also X1.1; no longer J2.1
Routing:
- net GND: track 137.3 -> 321.4 mm, vias 2 -> 5
- net CHARGER_VUSB_FIL: track 26.2 -> 73.5 mm, vias 1 -> 2
- net AGND: track 3.50 -> 46.6 mm, vias 0 -> 4
- net +3V3: track 43.2 -> 77.3 mm
- net CHARGER_STAT1: track 0.00 -> 28.1 mm, vias 0 -> 2
- net CHARGER_STAT2: track 0.00 -> 26.5 mm, vias 0 -> 2
- net CHARGER_!PG!: track 0.00 -> 25.9 mm, vias 0 -> 1
- net VDDCORE: track 0.00 -> 12.1 mm
- net CHARGER_NTC: track 26.1 -> 16.6 mm, vias 0 -> 1
- net +3V3_ANA: track 0.00 -> 5.95 mm
- net VDDOUT: track 0.00 -> 5.74 mm
- net BUCK_LX: track 6.25 -> 1.57 mm
- net XIN32: track 0.00 -> 4.37 mm
- net XOUT32: track 0.00 -> 4.28 mm
- net VBAT: track 12.3 -> 16.1 mm
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
Commit message: Senor Pinout refactored
Parts:
- moved JP1 315.6 mm to (74.0, 31.0), turned to 180 degrees
- moved JP2 312.6 mm to (74.0, 35.0), turned to 180 degrees
- moved JP7 306.2 mm to (74.0, 22.5)
- moved JP6 304.5 mm to (74.0, 27.0)
- moved JP4 295.1 mm to (64.0, 31.0), turned to 90 degrees
- moved JP5 292.2 mm to (62.7, 27.0)
- moved JP3 280.5 mm to (64.0, 22.6), turned to 90 degrees
- moved R21 196.1 mm to (-31.1, 83.3)
- moved R22 196.1 mm to (-31.1, 81.3)
- moved R23 196.1 mm to (-31.1, 79.2)
- moved R24 196.1 mm to (-31.1, 77.2)
- moved R25 196.1 mm to (-31.1, 75.2)
- moved R26 196.1 mm to (-31.1, 73.1)
- moved R27 196.1 mm to (-31.1, 71.0)
- moved R28 196.1 mm to (-31.1, 69.0)
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Connections:
- net !RESET!: now also U$1.3; no longer U$1.9
- net +3V3: now also U$1.5; no longer U$1.1
- net GND: now also U$1.7, U$1.9; no longer U$1.2, U$1.4
- net SENSOR_EN_0: now also IC8.27; no longer IC8.17
- net SENSOR_EN_1: now also IC8.23; no longer IC8.18
- net SENSOR_EN_2: now also IC8.21; no longer IC8.19
- net SENSOR_EN_3: now also IC8.19; no longer IC8.20
- net SENSOR_EN_4: now also IC8.17; no longer IC8.21
- net SENSOR_EN_5: now also IC8.28; no longer IC8.22
- net SENSOR_EN_6: now also IC8.26; no longer IC8.23
- net SENSOR_EN_7: now also IC8.22; no longer IC8.27
- net SENSOR_EN_8: now also IC8.20; no longer IC8.28
- net SENSOR_EN_9: now also IC8.18; no longer IC8.29
- net SENSOR_INT_0: now also IC8.34; no longer IC8.30
- net SENSOR_INT_1: now also IC8.32; no longer IC8.31
- net SENSOR_INT_2: now also IC8.30; no longer IC8.32
- net SENSOR_INT_3: now also IC8.16; no longer IC8.33
- net SENSOR_INT_4: now also IC8.14; no longer IC8.34
- net SENSOR_INT_5: now also IC8.33; no longer IC8.35
- net SENSOR_INT_6: now also IC8.31; no longer IC8.13
- net SENSOR_INT_7: now also IC8.29; no longer IC8.14
- net SENSOR_INT_9: now also IC8.13; no longer IC8.16
- net SENSOR_IN_0: now also IC8.9; no longer IC8.99
- net SENSOR_IN_1: now also IC8.7; no longer IC8.100
- net SENSOR_IN_2: now also IC8.5; no longer IC8.3
- net SENSOR_IN_3: now also IC8.3; no longer IC8.4
- net SENSOR_IN_4: now also IC8.99; no longer IC8.5
- net SENSOR_IN_5: now also IC8.10; no longer IC8.6
- net SENSOR_IN_6: now also IC8.8; no longer IC8.7
- net SENSOR_IN_7: now also IC8.6; no longer IC8.8
- net SENSOR_IN_8: now also IC8.4; no longer IC8.9
- net SENSOR_IN_9: now also IC8.100; no longer IC8.10
- net SWDCLK: now also U$1.2; no longer U$1.5
- net SWDIO: now also U$1.1; no longer U$1.3
Routing:
- net !RESET!: track 6.50 -> 76.4 mm
- net SWDIO: track 0.00 -> 31.5 mm
- net SWDCLK: track 0.00 -> 31.3 mm
- net USB_D_FIL_P: track 3.75 -> 20.8 mm
- net USB_D_FIL_N: track 3.91 -> 20.8 mm
- net GND: track 321.4 -> 325.4 mm
