File: pcb/circuit.brd (EAGLE design)
At the start: 80 x 80 mm, 148 parts, among them IC1 MCP1612-ADJI/MS, IC2 MCP73833-AMI/UN-ND, IC3 WE-TVS, IC4 MCP3423, IC5 ATWINC1510-MR210PB1952-ND, IC6 MAX3378EEUD, IC7 RN4870, IC8 ATSAML22N18A, J1 22-05-7038-03, J2 22-05-7038-03, Q1 ECX-1210, T1 PMOS, T10 NMOSSOT323, T11 NMOSSOT323, T12 NMOSSOT323, T2 NMOSSOT323, T3 NMOSSOT323, T4 NMOSSOT323, T5 NMOSSOT323, T6 NMOSSOT323, T7 NMOSSOT323, T8 NMOSSOT323, T9 NMOSSOT323, X1 USB2-MICRO, X10 2.5MM-AUDIO-JACK-MONONO_DRILL, X11 2.5MM-AUDIO-JACK-MONONO_DRILL, X12 2.5MM-AUDIO-JACK-MONONO_DRILL, X13 2.5MM-AUDIO-JACK-MONONO_DRILL, X14 MOLEX_1MM_FPC, X15 IGRID-20, X2 B3S-1000, X4 2.5MM-AUDIO-JACK-MONODRILL, X5 2.5MM-AUDIO-JACK-MONODRILL, X6 2.5MM-AUDIO-JACK-MONODRILL, X7 2.5MM-AUDIO-JACK-MONODRILL, X8 2.5MM-AUDIO-JACK-MONODRILL, X9 2.5MM-AUDIO-JACK-MONONO_DRILL

Commit message: routed sensor 0,1,5,6
Parts:
- moved J2 70.6 mm to (66.3, 22.8), turned to 90 degrees
- moved R21 59.9 mm to (10.1, 39.9), flipped to the top, turned to 90 degrees
- moved R22 59.9 mm to (12.1, 39.9), flipped to the top, turned to 90 degrees
- moved R24 58.7 mm to (14.2, 39.9), flipped to the top, turned to 90 degrees
- moved R26 57.8 mm to (16.2, 39.9), flipped to the top, turned to 270 degrees
- moved R28 57.3 mm to (18.2, 39.9), flipped to the top, turned to 90 degrees
- moved R34 56.7 mm to (9.05, 45.4), flipped to the top, turned to 270 degrees
- moved R23 55.7 mm to (13.1, 45.4), flipped to the top, turned to 90 degrees
- moved R25 55.0 mm to (15.2, 45.4), flipped to the top, turned to 90 degrees
- moved R27 54.7 mm to (17.2, 45.4), flipped to the top, turned to 90 degrees
- moved JP7 26.4 mm to (62.0, 46.0), flipped to the bottom
- moved JP6 24.0 mm to (73.0, 51.0), flipped to the bottom
- moved JP5 24.0 mm to (62.7, 51.0), flipped to the bottom, turned to 180 degrees
- moved JP3 19.4 mm to (58.0, 41.0), flipped to the bottom, turned to 270 degrees
- moved JP2 11.0 mm to (73.0, 46.0), flipped to the bottom, turned to 0 degrees
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Routing:
- net GND: track 325.4 -> 246.0 mm, vias 5 -> 6
- net SENSOR_IN_5: track 5.16 -> 60.3 mm, vias 0 -> 4
- net SENSOR_IN_0: track 5.16 -> 52.6 mm, vias 0 -> 3
- net SENSOR_INT_0: track 0.00 -> 42.3 mm, vias 0 -> 1
- net SENSOR_INT_6: track 0.00 -> 41.2 mm, vias 0 -> 2
- net SENSOR_INT_1: track 0.00 -> 35.7 mm, vias 0 -> 1
- net SENSOR_EN_5: track 9.61 -> 42.6 mm, vias 0 -> 2
- net SENSOR_INT_5: track 0.00 -> 32.6 mm
- net SWDIO: track 31.5 -> 0.00 mm
- net SWDCLK: track 31.3 -> 0.00 mm
- net SENSOR_EN_0: track 9.61 -> 40.9 mm, vias 0 -> 3
- net !RESET!: track 76.4 -> 56.4 mm
- net SENSOR_EN_1: track 9.68 -> 26.3 mm, vias 0 -> 1
- net SENSOR_EN_6: track 9.61 -> 24.9 mm, vias 0 -> 1
- net USB_D_FIL_P: track 20.8 -> 10.8 mm
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Other:
- board size 80 x 80 mm -> 80 x 70 mm
