File: pcb/circuit.sch (EAGLE design)
At the start: 148 parts, among them IC1 MCP1612-ADJI/MS, IC2 MCP73833-AMI/UN-ND, IC3 WE-TVS, IC4 MCP3423, IC5 ATWINC1510-MR210PB1952-ND, IC6 MAX3378EEUD, IC7 RN4870, IC8 ATSAML22N18A, J1 22-05-7038-03, J2 22-05-7038-03, Q1 ECX-1210, T1 PMOS, T10 NMOSSOT323, T11 NMOSSOT323, T12 NMOSSOT323, T2 NMOSSOT323, T3 NMOSSOT323, T4 NMOSSOT323, T5 NMOSSOT323, T6 NMOSSOT323, T7 NMOSSOT323, T8 NMOSSOT323, T9 NMOSSOT323, X1 USB2-MICRO, X10 2.5MM-AUDIO-JACK-MONONO_DRILL, X11 2.5MM-AUDIO-JACK-MONONO_DRILL, X12 2.5MM-AUDIO-JACK-MONONO_DRILL, X13 2.5MM-AUDIO-JACK-MONONO_DRILL, X14 MOLEX_1MM_FPC, X15 IGRID-20, X2 B3S-1000, X4 2.5MM-AUDIO-JACK-MONODRILL, X5 2.5MM-AUDIO-JACK-MONODRILL, X6 2.5MM-AUDIO-JACK-MONODRILL, X7 2.5MM-AUDIO-JACK-MONODRILL, X8 2.5MM-AUDIO-JACK-MONODRILL, X9 2.5MM-AUDIO-JACK-MONONO_DRILL

Commit message: started routing ATWINC
Parts:
- removed JP2: (no value), thermo:JP4
- added JP8: (no value), thermo:JP3
Connections:
- net !OLED_SPI_CS: now also JP8.3; no longer JP2.3
- net MISO_NC: no longer JP2.4
- net OLED_SPI_MOSI: now also JP8.1; no longer JP2.1
- net OLED_SPI_SCLK: now also JP8.2; no longer JP2.2
Changed lines of the file:
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@@
 <part name="JP6" library="thermo" deviceset="JP4" device=""/>
 <part name="JP7" library="thermo" deviceset="JP4" device=""/>
-<part name="JP2" library="thermo" deviceset="JP4" device=""/>
 <part name="JP1" library="thermo" deviceset="JP4" device=""/>
 <part name="U$1" library="thermo" deviceset="JTAG-EDGE-CON" device=""/>
+<part name="JP8" library="thermo" deviceset="JP3" device=""/>
 </parts>
 <sheets>
@@
 <instance part="JP6" gate="G$1" x="63.5" y="30.48" rot="R270"/>
 <instance part="JP7" gate="G$1" x="63.5" y="15.24" rot="R270"/>
-<instance part="JP2" gate="G$1" x="27.94" y="40.64" rot="R270"/>
 <instance part="JP1" gate="G$1" x="27.94" y="53.34" rot="R270"/>
+<instance part="JP8" gate="1" x="27.94" y="40.64" rot="R270"/>
 </instances>
 <busses>
@@
 <segment>
 <label x="22.86" y="43.18" size="0.889" layer="95" rot="R180" xref="yes"/>
-<pinref part="JP2" gate="G$1" pin="1"/>
+<pinref part="JP8" gate="1" pin="1"/>
 <wire x1="22.86" y1="43.18" x2="25.4" y2="43.18" width="0.1524" layer="91"/>
 </segment>
@@
 <segment>
 <label x="22.86" y="40.64" size="0.889" layer="95" rot="R180" xref="yes"/>
-<pinref part="JP2" gate="G$1" pin="2"/>
+<pinref part="JP8" gate="1" pin="2"/>
 <wire x1="22.86" y1="40.64" x2="25.4" y2="40.64" width="0.1524" layer="91"/>
 </segment>
@@
 <segment>
 <label x="22.86" y="38.1" size="0.889" layer="95" rot="R180" xref="yes"/>
-<pinref part="JP2" gate="G$1" pin="3"/>
+<pinref part="JP8" gate="1" pin="3"/>
 <wire x1="22.86" y1="38.1" x2="25.4" y2="38.1" width="0.1524" layer="91"/>
 </segment>
@@
 </segment>
 </net>
-<net name="MISO_NC" class="0">
-<segment>
-<label x="22.86" y="35.56" size="0.889" layer="95" rot="R180" xref="yes"/>
-<pinref part="JP2" gate="G$1" pin="4"/>
-<wire x1="22.86" y1="35.56" x2="25.4" y2="35.56" width="0.1524" layer="91"/>
-</segment>
-</net>
